File: dirty-ardscsino.kicad_pcb (KiCad board)
At the start: 2 copper layers, 42.7 x 75.2 mm, 15 parts, among them J1 SCSI, J2 Ext. Power (Unused), J3 DM3AT-SF-PEJM5, U1 STM32 Bluepill

Commit message: Add a smaller bypass to the termination grid as well
Parts:
- added C2: 0.1µF, Capacitor_SMD:C_0805_2012Metric_Pad1.15x1.40mm_HandSolder, F.Cu at (145.3, 149.6)
Routing:
- net Net-(C2-Pad2): track 119.7 -> 126.2 mm
- net Net-(C2-Pad1): track 108.2 -> 111.0 mm
Changed lines of the file:
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@@
     (thickness 1.6)
     (drawings 52)
-    (tracks 344)
+    (tracks 349)
     (zones 0)
-    (modules 15)
+    (modules 16)
     (nets 48)
   )
@@
   (net 43 "Net-(J3-Pad1)")
   (net 44 +5V)
-  (net 45 "Net-(JP2-Pad1)")
-  (net 46 "Net-(JP3-Pad1)")
-  (net 47 "Net-(U1-PadPC13)")
+  (net 45 "Net-(U1-PadPC13)")
+  (net 46 "Net-(C2-Pad2)")
+  (net 47 "Net-(C2-Pad1)")
   (net_class Default "This is the default net class."
     (clearance 0.2)
@@
     (add_net /TERM_POWER)
     (add_net GND)
+    (add_net "Net-(C2-Pad1)")
+    (add_net "Net-(C2-Pad2)")
     (add_net "Net-(J1-Pad25)")
     (add_net "Net-(J2-Pad2)")
@@
     (add_net "Net-(J3-PadSWA)")
     (add_net "Net-(J3-PadSWB)")
-    (add_net "Net-(JP2-Pad1)")
-    (add_net "Net-(JP3-Pad1)")
     (add_net "Net-(U1-PadNRST)")
     (add_net "Net-(U1-PadPA0)")
@@
     (add_net "Net-(U1-PadPC15)")
     (add_net "Net-(U1-PadVBAT)")
+  )
+  (module Capacitor_SMD:C_0805_2012Metric_Pad1.15x1.40mm_HandSolder (layer F.Cu)
+    (at 145.288 149.606)
+    (descr "Capacitor SMD 0805 (2012 Metric), square (rectangular) end terminal, IPC_7351 nominal with elongated pad for handsoldering. (Body size source: https://docs.google.com/spreadsheets/d/1BsfQQcO9C6DZCsRaXUlFlo91Tg2WpOkGARC1WS5S8t0/edit?usp=sharing), generated with kicad-footprint-generator")
+    (tags "capacitor handsolder")
+    (attr smd)
+    (fp_text reference C2 (at -3.302 0.254) (layer F.SilkS)
+      (effects (font (size 1 1) (thickness 0.15)))
+    )
+    (fp_text value 0.1µF (at 0 1.65) (layer F.Fab)
+      (effects (font (size 1 1) (thickness 0.15)))
+    )
+    (fp_text user %R (at 0 0) (layer F.Fab)
+      (effects (font (size 0.5 0.5) (thickness 0.08)))
+    )
+    (fp_line (start 1.85 0.95) (end -1.85 0.95) (layer F.CrtYd) (width 0.05))
+    (fp_line (start 1.85 -0.95) (end 1.85 0.95) (layer F.CrtYd) (width 0.05))
+    (fp_line (start -1.85 -0.95) (end 1.85 -0.95) (layer F.CrtYd) (width 0.05))
+    (fp_line (start -1.85 0.95) (end -1.85 -0.95) (layer F.CrtYd) (width 0.05))
+    (fp_line (start -0.261252 0.71) (end 0.261252 0.71) (layer F.SilkS) (width 0.12))
+    (fp_line (start -0.261252 -0.71) (end 0.261252 -0.71) (layer F.SilkS) (width 0.12))
+    (fp_line (start 1 0.6) (end -1 0.6) (layer F.Fab) (width 0.1))
+    (fp_line (start 1 -0.6) (end 1 0.6) (layer F.Fab) (width 0.1))
+    (fp_line (start -1 -0.6) (end 1 -0.6) (layer F.Fab) (width 0.1))
+    (fp_line (start -1 0.6) (end -1 -0.6) (layer F.Fab) (width 0.1))
+    (pad 2 smd roundrect (at 1.025 0) (size 1.15 1.4) (layers F.Cu F.Paste F.Mask) (roundrect_rratio 0.217391)
+      (net 46 "Net-(C2-Pad2)"))
+    (pad 1 smd roundrect (at -1.025 0) (size 1.15 1.4) (layers F.Cu F.Paste F.Mask) (roundrect_rratio 0.217391)
+      (net 47 "Net-(C2-Pad1)"))
+    (model ${KISYS3DMOD}/Capacitor_SMD.3dshapes/C_0805_2012Metric.wrl
+      (at (xyz 0 0 0))
+      (scale (xyz 1 1 1))
+      (rotate (xyz 0 0 0))
+    )
   )
   (module Connector_PinHeader_2.54mm:PinHeader_1x02_P2.54mm_Vertical (layer F.Cu)
@@
       (net 44 +5V))
     (pad 1 thru_hole rect (at 0 0 180) (size 1.7 1.7) (drill 1) (layers *.Cu *.Mask)
-      (net 46 "Net-(JP3-Pad1)"))
+      (net 46 "Net-(C2-Pad2)"))
     (model ${KISYS3DMOD}/Connector_PinHeader_2.54mm.3dshapes/PinHeader_1x02_P2.54mm_Vertical.wrl
       (at (xyz 0 0 0))
@@
       (net 2 GND))
     (pad 1 thru_hole rect (at 0 0 180) (size 1.7 1.7) (drill 1) (layers *.Cu *.Mask)
-      (net 45 "Net-(JP2-Pad1)"))
+      (net 47 "Net-(C2-Pad1)"))
     (model ${KISYS3DMOD}/Connector_PinHeader_2.54mm.3dshapes/PinHeader_1x02_P2.54mm_Vertical.wrl
       (at (xyz 0 0 0))
@@
     (descr "CP, Radial series, Radial, pin pitch=2.00mm, , diameter=5mm, Electrolytic Capacitor")
     (tags "CP Radial series Radial pin pitch 2.00mm  diameter 5mm Electrolytic Capacitor")
-    (fp_text reference C1 (at 4.318 -2.286) (layer F.SilkS)
+    (fp_text reference C1 (at 4.572 2.286) (layer F.SilkS)
       (effects (font (size 1 1) (thickness 0.15)))
     )
@@
       (net 33 "Net-(U1-PadPB1)"))
     (pad PC13 thru_hole circle (at 5.715 24.765 180) (size 1.524 1.524) (drill 0.762) (layers *.Cu *.Mask)
-      (net 47 "Net-(U1-PadPC13)"))
+      (net 45 "Net-(U1-PadPC13)"))
     (pad PC15 thru_hole circle (at 5.715 19.685 180) (size 1.524 1.524) (drill 0.762) (layers *.Cu *.Mask)
       (net 34 "Net-(U1-PadPC15)"))
@@
       (net 14 /SCSI_DBP))
     (pad 1 thru_hole rect (at 0 0 90) (size 1.6 1.6) (drill 0.8) (layers *.Cu *.Mask)
-      (net 46 "Net-(JP3-Pad1)"))
+      (net 46 "Net-(C2-Pad2)"))
     (model ${KISYS3DMOD}/Resistor_THT.3dshapes/R_Array_SIP10.wrl
       (at (xyz 0 0 0))
@@
       (net 14 /SCSI_DBP))
     (pad 1 thru_hole rect (at 0 0 90) (size 1.6 1.6) (drill 0.8) (layers *.Cu *.Mask)
-      (net 45 "Net-(JP2-Pad1)"))
+      (net 47 "Net-(C2-Pad1)"))
     (model ${KISYS3DMOD}/Resistor_THT.3dshapes/R_Array_SIP10.wrl
       (at (xyz 0 0 0))
@@
       (net 4 /SCSI_IO))
     (pad 1 thru_hole rect (at 0 0 270) (size 1.6 1.6) (drill 0.8) (layers *.Cu *.Mask)
-      (net 45 "Net-(JP2-Pad1)"))
+      (net 47 "Net-(C2-Pad1)"))
     (model ${KISYS3DMOD}/Resistor_THT.3dshapes/R_Array_SIP10.wrl
       (at (xyz 0 0 0))
@@
       (net 4 /SCSI_IO))
     (pad 1 thru_hole rect (at 0 0 270) (size 1.6 1.6) (drill 0.8) (layers *.Cu *.Mask)
-      (net 46 "Net-(JP3-Pad1)"))
+      (net 46 "Net-(C2-Pad2)"))
     (model ${KISYS3DMOD}/Resistor_THT.3dshapes/R_Array_SIP10.wrl
       (at (xyz 0 0 0))
@@
     (effects (font (size 1 1) (thickness 0.15)))
   )
-  (gr_text "ardSCSIno fork v0.1\nleadedsolder.com 2021" (at 148.336 149.86) (layer F.SilkS)
+  (gr_text "ardSCSIno fork v0.1\nleadedsolder.com 2021" (at 155.194 149.86) (layer F.SilkS)
     (effects (font (size 0.75 0.75) (thickness 0.15) italic))
   )
@@
   (segment (start 154.94 88.646) (end 154.94 78.232) (width 0.5) (layer B.Cu) (net 44) (status 10))
   (segment (start 163.195 77.978) (end 155.194 77.978) (width 0.5) (layer B.Cu) (net 44))
-  (segment (start 145.572 97.028) (end 144.272 97.028) (width 0.5) (layer F.Cu) (net 45) (status 20))
-  (segment (start 147.32 95.28) (end 145.572 97.028) (width 0.5) (layer F.Cu) (net 45))
-  (segment (start 147.32 91.186) (end 147.32 95.28) (width 0.5) (layer F.Cu) (net 45) (status 10))
-  (segment (start 144.272 79.63041) (end 144.272 97.028) (width 0.25) (layer B.Cu) (net 45) (status 20))
-  (segment (start 144.272 146.812) (end 139.992997 146.812) (width 0.25) (layer B.Cu) (net 45) (status 10))
-  (segment (start 135.324009 81.376989) (end 138.976998 77.724) (width 0.25) (layer B.Cu) (net 45))
-  (segment (start 139.992997 146.812) (end 135.324009 142.143012) (width 0.25) (layer B.Cu) (net 45))
-  (segment (start 135.324009 142.143012) (end 135.324009 81.376989) (width 0.25) (layer B.Cu) (net 45))
-  (segment (start 142.36559 77.724) (end 144.272 79.63041) (width 0.25) (layer B.Cu) (net 45))
-  (segment (start 138.976998 77.724) (end 142.36559 77.724) (width 0.25) (layer B.Cu) (net 45))
+  (segment (start 145.572 97.028) (end 144.272 97.028) (width 0.5) (layer F.Cu) (net 47) (status 20))
+  (segment (start 147.32 95.28) (end 145.572 97.028) (width 0.5) (layer F.Cu) (net 47))
+  (segment (start 147.32 91.186) (end 147.32 95.28) (width 0.5) (layer F.Cu) (net 47) (status 10))
+  (segment (start 144.272 79.63041) (end 144.272 97.028) (width 0.25) (layer B.Cu) (net 47) (status 20))
+  (segment (start 144.272 146.812) (end 139.992997 146.812) (width 0.25) (layer B.Cu) (net 47) (status 10))
+  (segment (start 135.324009 81.376989) (end 138.976998 77.724) (width 0.25) (layer B.Cu) (net 47))
+  (segment (start 139.992997 146.812) (end 135.324009 142.143012) (width 0.25) (layer B.Cu) (net 47))
+  (segment (start 135.324009 142.143012) (end 135.324009 81.376989) (width 0.25) (layer B.Cu) (net 47))
+  (segment (start 142.36559 77.724) (end 144.272 79.63041) (width 0.25) (layer B.Cu) (net 47))
+  (segment (start 138.976998 77.724) (end 142.36559 77.724) (width 0.25) (layer B.Cu) (net 47))
   (segment (start 150.876 91.186) (end 150.876 97.028) (width 0.5) (layer F.Cu) (net 46) (status 30))
   (segment (start 140.626587 148.082) (end 150.656 148.082) (width 0.25) (layer B.Cu) (net 46))
@@
   (segment (start 142.494 77.216) (end 138.848587 77.216) (width 0.25) (layer B.Cu) (net 46))
   (segment (start 144.78 79.502) (end 142.494 77.216) (width 0.25) (layer B.Cu) (net 46))
+  (segment (start 150.876 148.112) (end 150.876 146.812) (width 0.5) (layer F.Cu) (net 46))
+  (segment (start 149.382 149.606) (end 150.876 148.112) (width 0.5) (layer F.Cu) (net 46))
+  (segment (start 146.313 149.606) (end 149.382 149.606) (width 0.5) (layer F.Cu) (net 46))
+  (segment (start 144.263 146.821) (end 144.272 146.812) (width 0.5) (layer F.Cu) (net 47))
+  (segment (start 144.263 149.606) (end 144.263 146.821) (width 0.5) (layer F.Cu) (net 47))
   (zone (net 2) (net_name GND) (layer B.Cu) (hatch edge 0.508)
     (connect_pads (clearance 0.508))

Commit message: Move the cap so I don't hit it with USB
Parts:
- moved C1 8.67 mm to (156.9, 147.8)
Other:
- board text added: "#1"
- board text added: "ardSCSIno fork leadedsolder.com"
- board text added: "usb this end"
- board text added: "v0.1, 2021"
- board text removed: "ardSCSIno fork v0.1 leadedsolder.com 2021"
Changed lines of the file:
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@@
   (general
     (thickness 1.6)
-    (drawings 52)
-    (tracks 349)
+    (drawings 55)
+    (tracks 351)
     (zones 0)
     (modules 16)
@@
   )
   (module Capacitor_THT:CP_Radial_D5.0mm_P2.00mm (layer F.Cu)
-    (at 165.608 147.574 180)
+    (at 156.94 147.828 180)
     (descr "CP, Radial series, Radial, pin pitch=2.00mm, , diameter=5mm, Electrolytic Capacitor")
     (tags "CP Radial series Radial pin pitch 2.00mm  diameter 5mm Electrolytic Capacitor")
-    (fp_text reference C1 (at 4.572 2.286) (layer F.SilkS)
+    (fp_text reference C1 (at 2.508 3.556) (layer F.SilkS)
       (effects (font (size 1 1) (thickness 0.15)))
     )
@@
     )
   )
+  (gr_text "v0.1, 2021" (at 165.1 149.86) (layer F.SilkS)
+    (effects (font (size 1 1) (thickness 0.15)))
+  )
+  (gr_text "usb this end" (at 166.624 140.716) (layer F.SilkS)
+    (effects (font (size 1 1) (thickness 0.15)))
+  )
+  (gr_text "#1" (at 161.29 94.996) (layer F.SilkS)
+    (effects (font (size 1 1) (thickness 0.15)))
+  )
   (gr_text "files go here" (at 169.164 90.424) (layer F.SilkS)
     (effects (font (size 1 1) (thickness 0.15)))
@@
     (effects (font (size 1 1) (thickness 0.15)))
   )
-  (gr_text "ardSCSIno fork v0.1\nleadedsolder.com 2021" (at 155.194 149.86) (layer F.SilkS)
+  (gr_text "ardSCSIno fork\nleadedsolder.com" (at 164.846 147.828) (layer F.SilkS)
     (effects (font (size 0.75 0.75) (thickness 0.15) italic))
   )
@@
   (segment (start 138.537998 77.978) (end 142.494 77.978) (width 0.5) (layer F.Cu) (net 1))
   (segment (start 137.16 111.76) (end 134.874 109.474) (width 0.5) (layer F.Cu) (net 1) (status 10))
-  (via (at 175.006 89.789) (size 0.8) (drill 0.4) (layers F.Cu B.Cu) (net 44))
-  (segment (start 175.922001 98.397999) (end 175.922001 90.705001) (width 0.5) (layer F.Cu) (net 44))
-  (segment (start 175.922001 90.705001) (end 175.006 89.789) (width 0.5) (layer F.Cu) (net 44))
-  (segment (start 174.117 100.203) (end 175.922001 98.397999) (width 0.5) (layer F.Cu) (net 44) (status 10))
   (segment (start 163.022 77.806) (end 162.572 77.356) (width 0.5) (layer F.Cu) (net 2) (status 30))
   (segment (start 176.072 77.806) (end 163.022 77.806) (width 0.5) (layer F.Cu) (net 2) (status 30))
@@
   (segment (start 164.922 96.596) (end 165.227 96.901) (width 0.5) (layer F.Cu) (net 2))
   (segment (start 164.922 92.456) (end 164.922 96.596) (width 0.5) (layer F.Cu) (net 2) (status 10))
-  (segment (start 163.068 147.574) (end 163.608 147.574) (width 0.5) (layer B.Cu) (net 2) (status 30))
-  (segment (start 158.877 143.383) (end 163.068 147.574) (width 0.5) (layer B.Cu) (net 2) (status 30))
   (segment (start 158.877 140.843) (end 158.877 143.383) (width 0.5) (layer B.Cu) (net 2) (status 30))
+  (segment (start 154.94 146.69663) (end 154.94 147.828) (width 0.5) (layer B.Cu) (net 2))
+  (segment (start 154.94 146.24237) (end 154.94 146.69663) (width 0.5) (layer B.Cu) (net 2))
+  (segment (start 157.79937 143.383) (end 154.94 146.24237) (width 0.5) (layer B.Cu) (net 2))
+  (segment (start 158.877 143.383) (end 157.79937 143.383) (width 0.5) (layer B.Cu) (net 2))
   (segment (start 174.638761 141.930001) (end 175.768 140.800762) (width 0.25) (layer B.Cu) (net 3))
   (segment (start 169.968238 138.303) (end 173.595239 141.930001) (width 0.25) (layer B.Cu) (net 3))
@@
   (segment (start 160.528 113.792) (end 158.877 115.443) (width 0.25) (layer B.Cu) (net 35) (status 20))
   (segment (start 160.528 99.483238) (end 160.528 113.792) (width 0.25) (layer B.Cu) (net 35))
+  (via (at 175.006 89.789) (size 0.8) (drill 0.4) (layers F.Cu B.Cu) (net 44))
+  (segment (start 175.922001 98.397999) (end 175.922001 90.705001) (width 0.5) (layer F.Cu) (net 44))
+  (segment (start 175.922001 90.705001) (end 175.006 89.789) (width 0.5) (layer F.Cu) (net 44))
+  (segment (start 174.117 100.203) (end 175.922001 98.397999) (width 0.5) (layer F.Cu) (net 44) (status 10))
   (segment (start 154.94 78.232) (end 155.194 77.978) (width 0.5) (layer B.Cu) (net 44) (status 30))
   (segment (start 154.94 88.646) (end 150.876 88.646) (width 0.5) (layer B.Cu) (net 44) (status 30))
@@
   (segment (start 154.94 88.646) (end 154.94 78.232) (width 0.5) (layer B.Cu) (net 44) (status 10))
   (segment (start 163.195 77.978) (end 155.194 77.978) (width 0.5) (layer B.Cu) (net 44))
-  (segment (start 145.572 97.028) (end 144.272 97.028) (width 0.5) (layer F.Cu) (net 47) (status 20))
-  (segment (start 147.32 95.28) (end 145.572 97.028) (width 0.5) (layer F.Cu) (net 47))
-  (segment (start 147.32 91.186) (end 147.32 95.28) (width 0.5) (layer F.Cu) (net 47) (status 10))
-  (segment (start 144.272 79.63041) (end 144.272 97.028) (width 0.25) (layer B.Cu) (net 47) (status 20))
-  (segment (start 144.272 146.812) (end 139.992997 146.812) (width 0.25) (layer B.Cu) (net 47) (status 10))
-  (segment (start 135.324009 81.376989) (end 138.976998 77.724) (width 0.25) (layer B.Cu) (net 47))
-  (segment (start 139.992997 146.812) (end 135.324009 142.143012) (width 0.25) (layer B.Cu) (net 47))
-  (segment (start 135.324009 142.143012) (end 135.324009 81.376989) (width 0.25) (layer B.Cu) (net 47))
-  (segment (start 142.36559 77.724) (end 144.272 79.63041) (width 0.25) (layer B.Cu) (net 47))
-  (segment (start 138.976998 77.724) (end 142.36559 77.724) (width 0.25) (layer B.Cu) (net 47))
   (segment (start 150.876 91.186) (end 150.876 97.028) (width 0.5) (layer F.Cu) (net 46) (status 30))
   (segment (start 140.626587 148.082) (end 150.656 148.082) (width 0.25) (layer B.Cu) (net 46))
@@
   (segment (start 149.382 149.606) (end 150.876 148.112) (width 0.5) (layer F.Cu) (net 46))
   (segment (start 146.313 149.606) (end 149.382 149.606) (width 0.5) (layer F.Cu) (net 46))
+  (segment (start 145.572 97.028) (end 144.272 97.028) (width 0.5) (layer F.Cu) (net 47) (status 20))
+  (segment (start 147.32 95.28) (end 145.572 97.028) (width 0.5) (layer F.Cu) (net 47))
+  (segment (start 147.32 91.186) (end 147.32 95.28) (width 0.5) (layer F.Cu) (net 47) (status 10))
+  (segment (start 144.272 79.63041) (end 144.272 97.028) (width 0.25) (layer B.Cu) (net 47) (status 20))
+  (segment (start 144.272 146.812) (end 139.992997 146.812) (width 0.25) (layer B.Cu) (net 47) (status 10))
+  (segment (start 135.324009 81.376989) (end 138.976998 77.724) (width 0.25) (layer B.Cu) (net 47))
+  (segment (start 139.992997 146.812) (end 135.324009 142.143012) (width 0.25) (layer B.Cu) (net 47))
+  (segment (start 135.324009 142.143012) (end 135.324009 81.376989) (width 0.25) (layer B.Cu) (net 47))
+  (segment (start 142.36559 77.724) (end 144.272 79.63041) (width 0.25) (layer B.Cu) (net 47))
+  (segment (start 138.976998 77.724) (end 142.36559 77.724) (width 0.25) (layer B.Cu) (net 47))
   (segment (start 144.263 146.821) (end 144.272 146.812) (width 0.5) (layer F.Cu) (net 47))
   (segment (start 144.263 149.606) (end 144.263 146.821) (width 0.5) (layer F.Cu) (net 47))

Commit message: Add 180-degree floppy power conn
Parts:
- J2: value Ext. Power (Unused) -> 171825-4 (Ext. Power); footprint Connector_PinHeader_2.54mm:PinHeader_1x04_P2.54mm_Vertical -> 171825-4:TE_171825-4
- moved J2 0.80 mm to (155.4, 78.7), turned to 180 degrees
Connections:
- J2 pad 2: Net-(J2-Pad2) -> GND
- J2 pad 3: Net-(J2-Pad3) -> GND
- J2 pad 4: GND -> Net-(J2-Pad4)
Routing:
- net GND: track 86.8 -> 99.5 mm
