File: dirty-ardscsino.kicad_sch (KiCad schematic)
At the start: 16 parts, among them J1 SCSI, J2 171825-4 (Ext. Power), J3 DM3AT-SF-PEJM5, U1 STM32 Bluepill, U2 microSD-Breakout

Commit message: Convert LED to SMT; find parts for passives'
Parts:
- C2: LCSC (none) -> C28233
- D1: footprint LED_THT:LED_D3.0mm -> LED_SMD:LED_0805_2012Metric_Pad1.15x1.40mm_HandSolder; LCSC (none) -> C2292
- R1: value 560Ω -> 1kΩ; footprint Resistor_THT:R_Axial_DIN0207_L6.3mm_D2.5mm_P10.16mm_Horizontal -> Resistor_SMD:R_0805_2012Metric_Pad1.20x1.40mm_HandSolder; LCSC (none) -> C11702
Other:
- note added: "LED"
- note removed: "Optional external LED header"
- note removed: "Still not 100% sure about these SD card pinouts"
Changed lines of the file:
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@@
 		)
 	)
-	(text "Optional external LED header"
+	(text "LED"
 		(exclude_from_sim no)
-		(at 215.265 17.78 0)
+		(at 202.565 17.78 0)
 		(effects
 			(font
@@
 		)
 	)
-	(text "Still not 100% sure about these SD card pinouts"
-		(exclude_from_sim no)
-		(at 65.405 193.675 0)
-		(effects
-			(font
-				(size 1.27 1.27)
-			)
-			(justify left bottom)
-		)
-	)
 	(junction
 		(at 123.825 43.18)
@@
 			)
 		)
-		(property "LCSC" ""
+		(property "LCSC" "C28233"
 			(at 200.66 95.885 90)
 			(effects
@@
 			)
 		)
-		(property "Value" "560Ω"
+		(property "Value" "1kΩ"
 			(at 226.06 24.13 90)
 			(effects
@@
 			)
 		)
-		(property "Footprint" "Resistor_THT:R_Axial_DIN0207_L6.3mm_D2.5mm_P10.16mm_Horizontal"
+		(property "Footprint" "Resistor_SMD:R_0805_2012Metric_Pad1.20x1.40mm_HandSolder"
 			(at 226.06 27.94 0)
 			(effects
@@
 			)
 		)
+		(property "LCSC" "C11702"
+			(at 226.06 27.94 90)
+			(effects
+				(font
+					(size 1.27 1.27)
+				)
+				(hide yes)
+			)
+		)
 		(pin "2"
 		)
@@
 			)
 		)
-		(property "Footprint" "LED_THT:LED_D3.0mm"
+		(property "Footprint" "LED_SMD:LED_0805_2012Metric_Pad1.15x1.40mm_HandSolder"
 			(at 215.265 27.94 90)
 			(effects
@@
 			(at 215.265 27.94 0)
 			(effects
+				(font
+					(size 1.27 1.27)
+				)
+				(hide yes)
+			)
+		)
+		(property "LCSC" "C2292"
+			(at 215.265 27.94 0)
+			(effects

Commit message: discrete resistors
Parts:
- removed RN1, RN4: 220Ω, Resistor_THT:R_Array_SIP10, symbol Device:R_Network09_US
- removed RN2, RN3: 330Ω, Resistor_THT:R_Array_SIP10, symbol Device:R_Network09_US
- added R10, R11, R12, R13, R14, R15, R16, R17, R18, R19, R2, R20, R21, R22, R23, R24, R25, R26, R27, R28, R29, R3, R30, R31, R32, R33, R34, R35, R36, R37, R4, R5, R6, R7, R8, R9: R_Small_US, Resistor_SMD:R_0805_2012Metric_Pad1.20x1.40mm_HandSolder, symbol Device:R_Small_US
Connections:
- net GND: now also JP2.2 (B); no longer JP2.1 (A)
- net SCSI_ACK: now also R26.1, R8.2
- net SCSI_ATN: now also R10.2, R28.1
- net SCSI_BSY: now also R27.1, R9.2
- net SCSI_CD: now also R22.1, R4.2
- net SCSI_DAT0: now also R12.2, R30.1
- net SCSI_DAT1: now also R13.2, R31.1
- net SCSI_DAT2: now also R14.2, R32.1
- net SCSI_DAT3: now also R15.2, R33.1
- net SCSI_DAT4: now also R16.2, R34.1
- net SCSI_DAT5: now also R17.2, R35.1
- net SCSI_DAT6: now also R18.2, R36.1
- net SCSI_DAT7: now also R19.2, R37.1
- net SCSI_DBP: now also R11.2, R29.1
- net SCSI_IO: now also R2.2, R20.1
- net SCSI_MSG: now also R24.1, R6.2
- net SCSI_REQ: now also R21.1, R3.2
- net SCSI_RST: now also R25.1, R7.2
- net SCSI_SEL: now also R23.1, R5.2
- net at C2.2, JP3.2 (B): now also R10.1, R11.1, R12.1, R13.1, R14.1, R15.1, R16.1, R17.1, R18.1, R19.1, R2.1, R3.1, R4.1, R5.1, R6.1, R7.1, R8.1, R9.1
- net at C2.1: now also JP2.1 (A), R20.2, R21.2, R22.2, R23.2, R24.2, R25.2, R26.2, R27.2, R28.2, R29.2, R30.2, R31.2, R32.2, R33.2, R34.2, R35.2, R36.2, R37.2; no longer JP2.2 (B)
Other:
- note added: "220µF"
- note added: "330µF"
- note added: "TODO: assign values, footprints, LCSC number, put on board"
- note added: "TODO: is there an SMD version of this?"
- note added: "Termination Resistors"
- moved on the sheet: C2, JP2, JP3
