File: dirty-ardscsino.kicad_sch (KiCad schematic)
At the start: 19 parts, among them J1 SCSI, J2 171825-4 (Ext. Power), J3 DM3AT-SF-PEJM5, U1 STM32 Bluepill, U2 microSD-Breakout

Commit message: Bump cap to 10µF, label activity LED
Parts:
- C1: value 4.7µF -> 10µF
Changed lines of the file:
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@@
 			)
 		)
-		(property "Value" "4.7µF"
+		(property "Value" "10µF"
 			(at 130.175 28.9306 90)
 			(effects
